File: prusto_watch.kicad_pcb (KiCad board)
At the start: 2 copper layers, 37.4 x 37.4 mm, 54 parts, among them J1 USB_microB_2040002-1, J2 Conn_02x05_Odd_Even, J3 Vibration Motor, J4 Conn_01x06, J5 Conn_01x06, J6 Conn_02x03_Odd_Even, J7 Conn_02x03_Counter_Clockwise, Q3 RUM002N02T2L, SW2 SW_Push, U1 STM32F303RCT6-48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

Commit message: Update board layout
Parts:
- removed SW2: SW_Push, prusto_watch:PTS820_J15M_SMTR_LFS
- added R3: 10K, Resistors_SMD:R_0603, F.Cu at (152.7, 104.4)
- added REF***: KiCad-Logo2_6mm_SilkScreen, Symbols:KiCad-Logo2_6mm_SilkScreen, B.Cu at (146.3, 110.0)
- added REF***: OSHW-Logo2_7.3x6mm_SilkScreen, Symbols:OSHW-Logo2_7.3x6mm_SilkScreen, B.Cu at (140.7, 102.9)
- moved J2 11.2 mm to (132.3, 110.6), turned to 45 degrees
- moved R4 7.61 mm to (136.1, 93.2), turned to 180 degrees
- moved D1 7.39 mm to (136.1, 91.7), turned to 180 degrees
- moved BT1 6.61 mm to (128.5, 93.5), turned to 0 degrees
- moved R1 6.23 mm to (162.1, 99.6), turned to 90 degrees
- moved R16 5.00 mm to (137.2, 106.6)
- moved D2 4.68 mm to (163.8, 99.6)
- moved J5 4.12 mm to (153.0, 85.1)
- moved J1 3.94 mm to (128.9, 101.4)
- moved J7 3.64 mm to (163.8, 106.0)
- moved C6 3.45 mm to (133.6, 98.6)
- moved J3 3.10 mm to (163.6, 93.2)
- moved C15 2.96 mm to (141.5, 101.3), turned to 270 degrees
- moved FP1 2.90 mm to (153.3, 106.3)
- moved D4 2.84 mm to (142.2, 116.0)
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Connections:
- FP1 pad 16: /BLE_CONF -> (no net)
- U1 pad 30: /ACC_INT1 -> /CHRG_STAT
- U1 pad 31: /ACC_INT2 -> /ACC_INT1
- U1 pad 40: /BLE_CONF -> (no net)
- U1 pad 44: (no net) -> Net-(R3-Pad1)
- U3 pad 9: /ACC_INT2 -> (no net)
Routing:
- net +3V3: track 171.0 -> 151.9 mm, vias 4 -> 6
- net /BLE_CONF: track 15.5 -> 0.00 mm, vias 4 -> 0
- net /CHRG_STAT: track 1.39 -> 16.8 mm, vias 0 -> 2
- net GND: track 85.8 -> 99.6 mm, vias 35 -> 38
- net /ACC_INT2: track 13.8 -> 0.00 mm, vias 2 -> 0
- net /TMS: track 29.6 -> 17.3 mm
- net +5V: track 22.7 -> 14.0 mm
- net /TCK: track 26.0 -> 17.6 mm
- net /TDO: track 27.1 -> 18.8 mm
- net /DISP_SCS: track 21.9 -> 14.2 mm
- net /DISP_SDI: track 19.0 -> 11.7 mm
- net /DISP_SCLK: track 17.4 -> 10.2 mm
- net /TDI: track 25.5 -> 18.9 mm
- net /5V_EN: track 17.3 -> 10.9 mm
- net Net-(R3-Pad1): track 0.00 -> 5.45 mm
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Other:
- board text added: "+3V GND SCK CS SDO SDI"
- board text added: "B3 B2 GD B1 GD GD"
- board text added: "GND"
- board text added: "GND SCS SDI 5en +5V SCK"
- board text added: "PROG"
- board text added: "PWR"
- board text added: "Prusto Watch V0.4 Byron Wasti"
- board text added: "XX TX RX RS 3V GN"
